Commit message: pumaロボットとstanfordロボットのテンプレート作成

File: sushi_bot_description/urdf/sushi_bot/sushi_bot_macro.xacro (robot description, xacro)
@@ -1,7 +1,7 @@
 <?xml version="1.0" encoding="UTF-8"?>
 <robot xmlns:xacro="http://www.ros.org/wiki/xacro">
-  <xacro:include filename="$(find controlko_description)/urdf/common.xacro" />
+  <xacro:include filename="$(find sushi_bot_description)/urdf/common.xacro" />
   <!-- ※ *がついたパラメータはブロックパラメータ -->
-  <xacro:macro name="rrbot" params="prefix parent *origin">
+  <xacro:macro name="sushi_bot" params="prefix parent *origin">
     <!-- LINKS -->
     <!-- base link -->
@@ -9,14 +9,14 @@
       <xacro:default_inertial />
       <visual>
-        <origin xyz="0 0 0.15" rpy="0 0 0" />
+        <origin xyz="0 0 0.05" rpy="0 0 0" />
         <geometry>
-          <box size="0.3 0.3 0.3" />
+          <box size="0.3 0.3 0.1" />
         </geometry>
         <material name="StoglRobotics/Violet" />
       </visual>
       <collision>
-        <origin xyz="0 0 0.15" rpy="0 0 0" />
+        <origin xyz="0 0 0.05" rpy="0 0 0" />
         <geometry>
-          <box size="0.3 0.3 0.3" />
+          <box size="0.3 0.3 0.1" />
         </geometry>
       </collision>
@@ -92,5 +92,5 @@
     <!-- joint1 -->
     <joint name="${prefix}joint1" type="revolute">
-      <origin xyz="0 0 0.3" rpy="0 0 0" />
+      <origin xyz="0 0 0.1" rpy="0 0 0" />
       <parent link="${prefix}base_link" />
       <child link="${prefix}link1" />
