Commit message: 色の整理

File: sushi_bot_description/urdf/sushi_bot/simple_gripper_macro.xacro (robot description, xacro)
@@ -24,4 +24,7 @@
 			</collision>
 		</link>
+		<gazebo reference="${prefix}gripper_base">
+			<material>Gazebo/Grey</material>
+		</gazebo>
 		<!-- Right Finger -->
 		<joint name="${prefix}finger_right_joint" type="prismatic">
@@ -48,4 +51,7 @@
 			</collision>
 		</link>
+		<gazebo reference="${prefix}finger_right">
+			<material>Gazebo/White</material>
+		</gazebo>
 		<!-- Left Finger -->
 		<joint name="${prefix}finger_left_joint" type="prismatic">
@@ -72,4 +78,7 @@
 			</collision>
 		</link>
+		<gazebo reference="${prefix}finger_left">
+			<material>Gazebo/White</material>
+		</gazebo>
 		<joint name="${prefix}grasp_point_joint" type="fixed">
 			<parent link="${prefix}gripper_base" />

File: sushi_bot_description/urdf/sushi_bot/stanford_robot_macro.xacro (robot description, xacro)
@@ -14,5 +14,5 @@
           <box size="0.15 0.15 0.01" />
         </geometry>
-        <material name="Violet" />
+        <material name="Gray" />
       </visual>
       <collision>
@@ -24,5 +24,5 @@
     </link>
     <gazebo reference="${prefix}base_link">
-      <material>Gazebo/Orange</material>
+      <material>Gazebo/Grey</material>
     </gazebo>
     <joint name="${prefix}joint_1" type="revolute">
@@ -50,5 +50,5 @@
     </link>
     <gazebo reference="${prefix}link_0">
-      <material>Gazebo/Orange</material>
+      <material>Gazebo/Blue</material>
     </gazebo>
     <!-- Joint 2 Revolute about Y, between link_0 and link_1 -->
@@ -78,5 +78,5 @@
     </link>
     <gazebo reference="${prefix}link_1">
-      <material>Gazebo/Blue</material>
+      <material>Gazebo/Green</material>
     </gazebo>
     <!-- Joint 3 直動リンク Prismatic -->
@@ -106,5 +106,5 @@
     </link>
     <gazebo reference="${prefix}link_2">
-      <material>Gazebo/Yellow</material>
+      <material>Gazebo/Red</material>
     </gazebo>
     <!-- Joint 4 Revolute about Z, between link_2 and link_3 -->
@@ -134,5 +134,5 @@
     </link>
     <gazebo reference="${prefix}link_3">
-      <material>Gazebo/Green</material>
+      <material>Gazebo/Grey</material>
     </gazebo>
     <!-- Joint 5 Revolute about Y, between link_3 and link_4 -->
@@ -162,5 +162,5 @@
     </link>
     <gazebo reference="${prefix}link_4">
-      <material>Gazebo/Red</material>
+      <material>Gazebo/White</material>
     </gazebo>
     <!-- Joint 6 Revolute (wrist), between link_4 and flange -->
@@ -180,5 +180,5 @@
           <cylinder radius="0.025" length="0.01" />
         </geometry>
-        <material name="Black" />
+        <material name="Gray" />
       </visual>
       <collision>
@@ -190,5 +190,5 @@
     </link>
     <gazebo reference="${prefix}link_5">
-      <material>Gazebo/White</material>
+      <material>Gazebo/Black</material>
     </gazebo>
     <!-- 実機での作業点と一致するTOOLフレームの定義、エンドエフェクタ制御用フレーム -->
