Commit message: rvizで表示できた

File: sushi_bot_description/urdf/common.xacro (robot description, xacro)
@@ -82,3 +82,10 @@
     <emissive>0 0 0 0</emissive>
   </material>
+  <material name="Violet">
+    <color rgba="${102/255} ${46/255} ${145/255} 1.0" />
+    <ambient>1 0 0 1</ambient>
+    <diffuse>1 0 0 1</diffuse>
+    <specular>0.1 0.1 0.1 1</specular>
+    <emissive>0 0 0 0</emissive>
+  </material>
 </robot>

File: sushi_bot_description/urdf/sushi_bot.urdf.xacro (robot description, xacro)
@@ -6,8 +6,8 @@
   <xacro:arg name="sim_gazebo_classic" default="false" />
   <xacro:arg name="simulation_controllers" default="" />
-  <xacro:include filename="$(find sushi_bot_description)/urdf/sushi_bot/sushi_bot_macro.xacro" />
-  <xacro:include filename="$(find sushi_bot_description)/urdf/sushi_bot/puma_robot_macro.xacro" />
+  <!-- <xacro:include filename="$(find sushi_bot_description)/urdf/sushi_bot/sushi_bot_macro.xacro" />
+  <xacro:include filename="$(find sushi_bot_description)/urdf/sushi_bot/puma_robot_macro.xacro" /> -->
   <xacro:include filename="$(find sushi_bot_description)/urdf/sushi_bot/stanford_robot_macro.xacro" />
-  <xacro:include filename="$(find sushi_bot_description)/urdf/sushi_bot/sushi_bot_macro.ros2_control.xacro" />
+  <!-- <xacro:include filename="$(find sushi_bot_description)/urdf/sushi_bot/sushi_bot_macro.ros2_control.xacro" /> -->
   <!-- "world"に固定されたリンクを作る -->
   <link name="world" />

File: sushi_bot_description/urdf/sushi_bot/stanford_robot_macro.xacro (robot description, xacro)
@@ -17,5 +17,5 @@
           <box size="0.15 0.15 0.01" />
         </geometry>
-        <material name="StoglRobotics/Violet" />
+        <material name="Violet" />
       </visual>
       <collision>
@@ -195,40 +195,31 @@
       <material>Gazebo/White</material>
     </gazebo>
+    <!-- 実機での作業点と一致するTOOLフレームの定義、エンドエフェクタ制御用フレーム -->
+    <!-- 実体なし、TFツリーやMoveItとの整合のために非常に重要 -->
+    <link name="${prefix}tool0" />
     <!-- Flange Link -->
-    <link name="${prefix}flange_link">
-      <!-- <inertial>
-        <origin xyz="0 0 0.025" rpy="0 0 0" />
-        <mass value="0.1" />
-        <inertia ixx="0.001" ixy="0.0" ixz="0.0" iyy="0.001" iyz="0.0" izz="0.001" />
-      </inertial>
-      <visual>
-        <origin xyz="0 0 0.025" rpy="0 0 0" />
-        <geometry>
-          <cylinder radius="0.04" length="0.05" />
-        </geometry>
-        <material name="Cyan" />
-      </visual>
-      <collision>
-        <origin xyz="0 0 0.025" rpy="0 0 0" />
-        <geometry>
-          <cylinder radius="0.04" length="0.05" />
-        </geometry>
-      </collision> -->
-    </link>
-    <gazebo reference="${prefix}flange_link">
-      <material>Gazebo/Gray</material>
-    </gazebo>
-    <!-- Fixed tool0 link -->
-    <link name="${prefix}tool0">
-      <inertial>
-        <origin xyz="0 0 0" rpy="0 0 0" />
-        <mass value="0.01" />
-        <inertia ixx="0.0001" ixy="0.0" ixz="0.0" iyy="0.0001" iyz="0.0" izz="0.0001" />
-      </inertial>
-      <!-- Optional: small visual or collision geometry could be added here -->
-    </link>
-    <joint name="${prefix}tool0_fixed_joint" type="fixed">
-      <parent link="${prefix}flange_link" />
+    <!-- ツール（グリッパ、吸着パッドなど）を取り付ける標準フレーム -->
+    <!-- REP 103準拠でX+軸がツール取付方向（前方）を向く -->
+    <link name="${prefix}flange" />
+    <!-- 実機制御器とURDFの原点を一致させるための基準フレーム -->
+    <!-- ROS-I仕様の標準、制御器の「ベース」座標に対応 -->
+    <link name="${prefix}base" />
+    <!-- tool joint - fixed -->
+    <joint name="${prefix}tool_joint" type="fixed">
+      <parent link="${prefix}link_5" />
       <child link="${prefix}tool0" />
+      <origin xyz="0 0 0.01" rpy="0 ${-pi} ${pi/2}" />
+    </joint>
+    <!-- base joint - fixed -->
+    <joint name="${prefix}base_link-base_joint" type="fixed">
+      <origin xyz="0 0 0" rpy="0 0 0" />
+      <parent link="${prefix}base_link" />
+      <child link="${prefix}base" />
+    </joint>
+    <!-- flange joint - fixed -->
+    <joint name="${prefix}tool0-flange_joint" type="fixed">
+      <origin xyz="0 0 0" rpy="0 0 0" />
+      <parent link="${prefix}tool0" />
+      <child link="${prefix}flange" />
     </joint>
   </xacro:macro>
