Commit message: ハンド作成できた

File: sushi_bot_description/urdf/sushi_bot.urdf.xacro (robot description, xacro)
@@ -6,20 +6,14 @@
   <xacro:arg name="sim_gazebo_classic" default="false" />
   <xacro:arg name="simulation_controllers" default="" />
-  <!-- <xacro:include filename="$(find sushi_bot_description)/urdf/sushi_bot/sushi_bot_macro.xacro" />
-  <xacro:include filename="$(find sushi_bot_description)/urdf/sushi_bot/puma_robot_macro.xacro" /> -->
+  <xacro:include filename="$(find sushi_bot_description)/urdf/common.xacro" />
   <xacro:include filename="$(find sushi_bot_description)/urdf/sushi_bot/stanford_robot_macro.xacro" />
-  <!-- <xacro:include filename="$(find sushi_bot_description)/urdf/sushi_bot/sushi_bot_macro.ros2_control.xacro" /> -->
+  <xacro:include filename="$(find sushi_bot_description)/urdf/sushi_bot/simple_gripper_macro.xacro" />
   <!-- "world"に固定されたリンクを作る -->
   <link name="world" />
   <!-- ロボットのマクロを読み込む -->
-  <!-- <xacro:sushi_bot prefix="$(arg prefix)" parent="world">
-    <origin xyz="0 0 0" rpy="0 0 0" />
-  </xacro:sushi_bot> -->
   <xacro:stanford_robot prefix="$(arg prefix)" parent="world">
     <origin xyz="0 0 0" rpy="0 0 0" />
   </xacro:stanford_robot>
-  <!-- <xacro:puma_robot prefix="$(arg prefix)" parent="world">
-    <origin xyz="0 0 0" rpy="0 0 0" />
-  </xacro:puma_robot> -->
+  <xacro:simple_gripper prefix="$(arg prefix)" parent="$(arg prefix)tool0" />
   <!-- コントローラーのマクロを読み込む -->
   <!-- <xacro:sushi_bot_ros2_control

File: sushi_bot_description/urdf/sushi_bot/stanford_robot_macro.xacro (robot description, xacro)
@@ -1,5 +1,4 @@
 <?xml version="1.0" encoding="UTF-8"?>
 <robot xmlns:xacro="http://www.ros.org/wiki/xacro">
-  <xacro:include filename="$(find sushi_bot_description)/urdf/common.xacro" />
   <!-- ※ *がついたパラメータはブロックパラメータ -->
   <xacro:macro name="stanford_robot" params="prefix parent *origin">
@@ -209,5 +208,6 @@
       <parent link="${prefix}link_5" />
       <child link="${prefix}tool0" />
-      <origin xyz="0 0 0.01" rpy="0 ${-pi} ${pi/2}" />
+      <!-- <origin xyz="0 0 0.01" rpy="0 ${-pi} ${pi/2}" /> -->
+      <origin xyz="0 0 0.01" rpy="0 0 0" />
     </joint>
     <!-- base joint - fixed -->

Commit message: brigupパッケージ作成

File: sushi_bot_description/urdf/sushi_bot.urdf.xacro (robot description, xacro)
@@ -9,4 +9,5 @@
   <xacro:include filename="$(find sushi_bot_description)/urdf/sushi_bot/stanford_robot_macro.xacro" />
   <xacro:include filename="$(find sushi_bot_description)/urdf/sushi_bot/simple_gripper_macro.xacro" />
+  <xacro:include filename="$(find sushi_bot_description)/urdf/sushi_bot/sushi_bot_macro.ros2_control.xacro" />
   <!-- "world"に固定されたリンクを作る -->
   <link name="world" />
@@ -17,12 +18,12 @@
   <xacro:simple_gripper prefix="$(arg prefix)" parent="$(arg prefix)tool0" />
   <!-- コントローラーのマクロを読み込む -->
-  <!-- <xacro:sushi_bot_ros2_control
+  <xacro:sushi_bot_ros2_control
     name="sushi_bot"
     prefix="$(arg prefix)"
     use_mock_hardware="$(arg use_mock_hardware)"
     mock_sensor_commands="$(arg mock_sensor_commands)"
-    sim_gazebo_classic="$(arg sim_gazebo_classic)" /> -->
+    sim_gazebo_classic="$(arg sim_gazebo_classic)" />
   <!-- Gazebo Classicのプラグインを読み込む -->
-  <!-- <xacro:if value="$(arg sim_gazebo_classic)">
+  <xacro:if value="$(arg sim_gazebo_classic)">
     <gazebo reference="world">
     </gazebo>
@@ -32,4 +33,4 @@
       </plugin>
     </gazebo>
-  </xacro:if> -->
+  </xacro:if>
 </robot>

File: sushi_bot_description/urdf/sushi_bot/sushi_bot_macro.ros2_control.xacro (robot description, xacro)
@@ -1,11 +1,5 @@
 <?xml version="1.0" encoding="UTF-8"?>
 <robot xmlns:xacro="http://www.ros.org/wiki/xacro">
-  <!-- モックコンポーネントの設定 -->
-  <!-- The caret ^ indicates to use the outer-scope property (with same
-  name).
-   The pipe | indicates to use the given fallback if the property is not defined in outer scope. -->
-  <!-- `^`は，外部スコーププロパティ（同名）を使用します -->
-  <!-- `|`は，外部スコープでプロパティが定義されていない場合に指定されたフォールバックを使用します -->
-  <xacro:macro name="rrbot_ros2_control"
+  <xacro:macro name="sushi_bot_ros2_control"
     params="name
             prefix
@@ -24,10 +18,6 @@
           <plugin>gazebo_ros2_control/GazeboSystem</plugin>
         </xacro:if>
-        <!-- 自作のHardware Interface -->
-        <xacro:unless value="${use_mock_hardware or sim_gazebo_classic}">
-          <plugin>controlko_hardware_interface/RRBotHardwareInterface</plugin>
-        </xacro:unless>
       </hardware>
-      <joint name="${prefix}joint1">
+      <joint name="${prefix}joint_1">
         <command_interface name="position" />
         <command_interface name="velocity" />
@@ -42,5 +32,5 @@
         </state_interface>
       </joint>
-      <joint name="${prefix}joint2">
+      <joint name="${prefix}joint_2">
         <command_interface name="position" />
         <command_interface name="velocity" />
@@ -55,27 +45,78 @@
         </state_interface>
       </joint>
-      <!-- 6軸 Force-Torque-Sensor センサ -->
-      <sensor name="tcp_fts_sensor">
-        <state_interface name="fx" />
-        <state_interface name="fy" />
-        <state_interface name="fz" />
-        <state_interface name="tx" />
-        <state_interface name="ty" />
-        <state_interface name="tz" />
-        <param name="frame_id">tool0</param>
-      </sensor>
-      <!-- GPIO -->
-      <gpio name="flange_gpios">
-        <state_interface name="digital_input1" />
-        <state_interface name="digital_input2" />
-        <command_interface name="digital_output1">
-          <param name="initial_value">false</param>
-        </command_interface>
-        <!-- <state_interface name="digital_output1" /> -->
-        <command_interface name="digital_output2">
-          <param name="initial_value">false</param>
-        </command_interface>
-        <!-- <state_interface name="digital_output2" /> -->
-      </gpio>
+      <joint name="${prefix}joint_3">
+        <command_interface name="position" />
+        <command_interface name="velocity" />
+        <state_interface name="position">
+          <param name="initial_value">0.0</param>
+        </state_interface>
+        <state_interface name="velocity">
+          <param name="initial_value">0.0</param>
+        </state_interface>
+        <state_interface name="effort">
+          <param name="initial_value">0.0</param>
+        </state_interface>
+      </joint>
+      <joint name="${prefix}joint_4">
+        <command_interface name="position" />
+        <command_interface name="velocity" />
+        <state_interface name="position">
+          <param name="initial_value">0.0</param>
+        </state_interface>
+        <state_interface name="velocity">
+          <param name="initial_value">0.0</param>
+        </state_interface>
+        <state_interface name="effort">
+          <param name="initial_value">0.0</param>
+        </state_interface>
+      </joint>
+      <joint name="${prefix}joint_5">
+        <command_interface name="position" />
+        <command_interface name="velocity" />
+        <state_interface name="position">
+          <param name="initial_value">0.0</param>
+        </state_interface>
+        <state_interface name="velocity">
+          <param name="initial_value">0.0</param>
+        </state_interface>
+        <state_interface name="effort">
+          <param name="initial_value">0.0</param>
+        </state_interface>
+      </joint>
+      <joint name="${prefix}joint_6">
+        <command_interface name="position" />
+        <command_interface name="velocity" />
+        <state_interface name="position">
+          <param name="initial_value">0.0</param>
+        </state_interface>
+        <state_interface name="velocity">
+          <param name="initial_value">0.0</param>
+        </state_interface>
+        <state_interface name="effort">
+          <param name="initial_value">0.0</param>
+        </state_interface>
+      </joint>
+      <!-- Finger Left Joint -->
+      <joint name="${prefix}finger_left_joint">
+        <command_interface name="position" />
+        <command_interface name="effort" />
+        <state_interface name="position">
+          <param name="initial_value">0.0</param>
+        </state_interface>
+        <state_interface name="effort">
+          <param name="initial_value">0.0</param>
+        </state_interface>
+      </joint>
+      <!-- Finger Right Joint -->
+      <joint name="${prefix}finger_right_joint">
+        <command_interface name="position" />
+        <command_interface name="effort" />
+        <state_interface name="position">
+          <param name="initial_value">0.0</param>
+        </state_interface>
+        <state_interface name="effort">
+          <param name="initial_value">0.0</param>
+        </state_interface>
+      </joint>
     </ros2_control>
   </xacro:macro>
