Commit message: 誤字修正: Gray->Grey

File: controlko_description/urdf/rrbot/rrbot_macro.xacro (robot description, xacro)
@@ -67,5 +67,5 @@
     </link>
     <gazebo reference="${prefix}link2">
-      <material>Gazebo/Gray</material>
+      <material>Gazebo/Grey</material>
     </gazebo>
     <!-- 座標マーカー的な ~~~ -->

File: sushi_bot_description/urdf/common.xacro (robot description, xacro)
@@ -51,5 +51,5 @@
     <emissive>0 0 0 0</emissive>
   </material>
-  <material name="Gray">
+  <material name="Grey">
     <color rgba="${128/255} ${128/255} ${128/255} 1.0" />
     <ambient>0.5 0.5 0.5 1</ambient>

File: sushi_bot_description/urdf/sushi_bot/simple_gripper_macro.xacro (robot description, xacro)
@@ -15,5 +15,5 @@
 					<box size="0.04 0.05 0.01" />
 				</geometry>
-				<material name="Gray" />
+				<material name="Grey" />
 			</visual>
 			<collision>

File: sushi_bot_description/urdf/sushi_bot/stanford_robot_macro.xacro (robot description, xacro)
@@ -14,5 +14,5 @@
           <box size="0.15 0.15 0.01" />
         </geometry>
-        <material name="Gray" />
+        <material name="Grey" />
       </visual>
       <collision>
@@ -124,5 +124,5 @@
           <cylinder radius="0.025" length="0.04" />
         </geometry>
-        <material name="Gray" />
+        <material name="Grey" />
       </visual>
       <collision>
@@ -180,5 +180,5 @@
           <cylinder radius="0.025" length="0.01" />
         </geometry>
-        <material name="Gray" />
+        <material name="Grey" />
       </visual>
       <collision>
